File: hidpawx_hardware/hidpawx_hardware.kicad_pcb (KiCad board)
At the start: 2 copper layers, 60 x 69 mm, 22 parts, among them J1 NFC, J2 RELAY_INTERRUPT, K1 MAIN_RELAY, Q1 AO3400A, Q2 AO3400A, U1 ESP32-S3-DevKitC

Commit message: starting back up on this, need to learn how websockets work
Connections:
- net Net-(J2-Pin_1) renamed /MAINS_IN
- net Net-(J2-Pin_2) renamed /MAINS_OUT
Routing:
- net /MAINS_OUT: track 24.3 -> 48.8 mm
- net /MAINS_IN: track 10.5 -> 20.9 mm
- added copper zone on B.Cu, net /MAINS_IN
- added copper zone on F.Cu, net /MAINS_IN
- added copper zone on B.Cu, net /MAINS_OUT
- added copper zone on F.Cu, net /MAINS_OUT
Changed lines of the file:
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@@
 	(net 7 "/NFC_SCL")
 	(net 8 "/NFC_SDA")
-	(net 9 "Net-(J2-Pin_2)")
-	(net 10 "Net-(J2-Pin_1)")
+	(net 9 "/MAINS_OUT")
+	(net 10 "/MAINS_IN")
 	(net 11 "Net-(Q2-D)")
 	(net 12 "Net-(Q1-G)")
@@
 			(layers "*.Cu" "*.Mask")
 			(remove_unused_layers no)
-			(net 9 "Net-(J2-Pin_2)")
+			(net 9 "/MAINS_OUT")
 			(pintype "passive")
 		)
@@
 			(layers "*.Cu" "*.Mask")
 			(remove_unused_layers no)
-			(net 10 "Net-(J2-Pin_1)")
+			(net 10 "/MAINS_IN")
 			(pintype "passive")
 		)
@@
 			(layers "*.Cu" "*.Mask")
 			(remove_unused_layers no)
-			(net 10 "Net-(J2-Pin_1)")
+			(net 10 "/MAINS_IN")
 			(pinfunction "Pin_1")
 			(pintype "passive")
@@
 			(layers "*.Cu" "*.Mask")
 			(remove_unused_layers no)
-			(net 9 "Net-(J2-Pin_2)")
+			(net 9 "/MAINS_OUT")
 			(pinfunction "Pin_2")
 			(pintype "passive")
@@
 	)
 	(segment
+		(start 162 60.146288)
+		(end 158.299 56.445288)
+		(width 2.5)
+		(layer "B.Cu")
+		(net 9)
+	)
+	(segment
+		(start 162 74)
+		(end 162 60.146288)
+		(width 2.5)
+		(layer "B.Cu")
+		(net 9)
+	)
+	(segment
+		(start 158.299 56.445288)
+		(end 158.299 51.081904)
+		(width 2.5)
+		(layer "B.Cu")
+		(net 9)
+	)
+	(segment
 		(start 168 59.8)
 		(end 168 55.449304)
@@
 	)
 	(segment
+		(start 163.901 51.252)
+		(end 163.901 51.081904)
+		(width 2.5)
+		(layer "B.Cu")
+		(net 10)
+	)
+	(segment
+		(start 168 59.8)
+		(end 168 55.351)
+		(width 2.5)
+		(layer "B.Cu")
+		(net 10)
+	)
+	(segment
+		(start 168 55.351)
+		(end 163.901 51.252)
+		(width 2.5)
+		(layer "B.Cu")
+		(net 10)
+	)
+	(segment
 		(start 148 94)
 		(end 152.0125 94)
@@
 			)
 		)
+	)
+	(zone
+		(net 9)
+		(net_name "/MAINS_OUT")
+		(layers "F.Cu" "B.Cu")
+		(hatch edge 0.5)
+		(priority 1)
+		(connect_pads yes
+			(clearance 0.18)
+		)
+		(min_thickness 0.18)
+		(filled_areas_thickness no)
+		(fill yes
+			(thermal_gap 0.5)
+			(thermal_bridge_width 0.5)
+		)
+		(polygon
+			(pts
+				(xy 160 48.5) (xy 160 56.25) (xy 164 56.25) (xy 164 76) (xy 160 76) (xy 160 68) (xy 157.75 68) (xy 157.75 58.25)
+				(xy 156.5 56.75) (xy 156.5 48.5)
+			)
+		)
+	)
+	(zone
+		(net 10)
+		(net_name "/MAINS_IN")
+		(layers "F.Cu" "B.Cu")
+		(hatch edge 0.5)
+		(priority 2)
+		(connect_pads yes
+			(clearance 0.18)
+		)
+		(min_thickness 0.18)
+		(filled_areas_thickness no)
+		(fill yes
+			(thermal_gap 0.5)
+			(thermal_bridge_width 0.5)
+		)
+		(polygon
+			(pts
+				(xy 162.25 48.5) (xy 162.25 54.5) (xy 166.25 54.5) (xy 166.25 61.75) (xy 170 61.75) (xy 170 48.5)
+			)
+		)
