File: hidpawx_hardware/hidpawx_hardware.kicad_sch (KiCad schematic)
At the start: 20 parts, among them J1 NFC, J2 RELAY_INTERRUPT, K1 MAIN_RELAY, Q1 AO3400A, Q2 AO3400A, U1 ESP32-S3-DevKitC

Commit message: starting back up on this, need to learn how websockets work
Connections:
- net MAINS_OUT: now reaches J2.2 (Pin_2), K1.11
- net MAINS_IN: now reaches J2.1 (Pin_1), K1.14
Changed lines of the file:
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@@
+		)
+	)
+	(label "MAINS_OUT"
+		(at 156.21 52.07 0)
+		(effects
+			(font
+				(size 1.27 1.27)
+			)
+			(justify left bottom)
 		)
 	)
@@
 		(effects
 			(font
+				(size 1.27 1.27)
+			)
+			(justify left bottom)
+		)
+	)
+	(label "MAINS_IN"
+		(at 156.21 49.53 0)
+		(effects
+			(font
